File: POxiM-fingersensor.kicad_pcb (KiCad board)
At the start: 2 copper layers, 10 x 36.5 mm, 5 parts, among them J3 To readout unit

Commit message: Rev F
Routing:
- net /LED.IR: track 25.5 -> 24.5 mm
- net /Photodiode: vias 0 -> 16
- net +5V: vias 0 -> 16
Other:
- board text added: "Finger sensor Rev F"
- board text removed: "Finger sensor Rev D"
Changed lines of the file:
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@@
     (thickness 1.6)
     (drawings 46)
-    (tracks 27)
+    (tracks 60)
     (zones 0)
     (modules 5)
@@
     (effects (font (size 1 1) (thickness 0.15)))
   )
-  (gr_poly (pts (xy 109.75 74.575) (xy 112.75 74.575) (xy 112.75 76.325) (xy 109.75 76.325)) (layer F.Mask) (width 0.55))
-  (gr_poly (pts (xy 105.25 74.575) (xy 108.25 74.575) (xy 108.25 76.325) (xy 105.25 76.325)) (layer F.Mask) (width 0.55))
+  (gr_poly (pts (xy 109.75 73.5) (xy 112.75 73.5) (xy 112.75 76.325) (xy 109.75 76.325)) (layer F.Mask) (width 0.55))
+  (gr_poly (pts (xy 105.25 73.5) (xy 107.75 73.5) (xy 108.25 74) (xy 108.25 76.325) (xy 105.25 76.325)) (layer F.Mask) (width 0.55))
   (gr_line (start 104 76.9) (end 114 76.9) (layer Edge.Cuts) (width 0.6))
   (gr_line (start 112 63.75) (end 114 63.75) (layer F.SilkS) (width 0.12))
@@
   (gr_line (start 104 76.9) (end 104 56.5) (layer Edge.Cuts) (width 0.6))
   (gr_line (start 114 76.9) (end 114 56.5) (layer Edge.Cuts) (width 0.6))
-  (gr_text "Finger sensor\nRev D" (at 109 85) (layer F.SilkS)
+  (gr_text "Finger sensor\nRev F" (at 109 85) (layer F.SilkS)
     (effects (font (size 0.8 0.8) (thickness 0.15)))
   )
@@
   (gr_arc (start 109.75 80.25) (end 109.75 79.75) (angle -90) (layer F.SilkS) (width 0.15))
   (gr_line (start 108.75 80.6) (end 109.25 80.6) (layer F.SilkS) (width 0.15))
-  (gr_poly (pts (xy 109.75 80.25) (xy 112.75 80.25) (xy 112.75 82) (xy 109.75 82)) (layer F.Mask) (width 0.55))
-  (gr_poly (pts (xy 105.25 80.25) (xy 108.25 80.25) (xy 108.25 82) (xy 105.25 82)) (layer F.Mask) (width 0.55))
+  (gr_poly (pts (xy 109.75 80.25) (xy 112.75 80.25) (xy 112.75 83) (xy 109.75 83)) (layer F.Mask) (width 0.55))
+  (gr_poly (pts (xy 105.25 80.25) (xy 108.25 80.25) (xy 108.25 83) (xy 105.25 83)) (layer F.Mask) (width 0.55))
   (gr_line (start 104 79) (end 114 79) (layer Edge.Cuts) (width 0.6))
   (gr_line (start 109 88.5) (end 109 89) (layer Cmts.User) (width 0.15))
@@
   (gr_line (start 104 93) (end 104 79) (layer Edge.Cuts) (width 0.6))
   (gr_line (start 104 93) (end 114 93) (layer Edge.Cuts) (width 0.6))
+  (via (at 105.25 74.75) (size 0.8) (drill 0.4) (layers F.Cu B.Cu) (net 1))
+  (via (at 108.25 74.75) (size 0.8) (drill 0.4) (layers F.Cu B.Cu) (net 1))
+  (via (at 108.25 76) (size 0.8) (drill 0.4) (layers F.Cu B.Cu) (net 1))
+  (via (at 106.75 76) (size 0.8) (drill 0.4) (layers F.Cu B.Cu) (net 1))
+  (via (at 107.5 75.375) (size 0.8) (drill 0.4) (layers F.Cu B.Cu) (net 1))
+  (via (at 106 75.375) (size 0.8) (drill 0.4) (layers F.Cu B.Cu) (net 1))
+  (via (at 112 75.375) (size 0.8) (drill 0.4) (layers F.Cu B.Cu) (net 2))
+  (via (at 109.75 76) (size 0.8) (drill 0.4) (layers F.Cu B.Cu) (net 2))
+  (via (at 112.75 74.75) (size 0.8) (drill 0.4) (layers F.Cu B.Cu) (net 2))
+  (via (at 112.75 76) (size 0.8) (drill 0.4) (layers F.Cu B.Cu) (net 2))
+  (via (at 110.5 75.375) (size 0.8) (drill 0.4) (layers F.Cu B.Cu) (net 2))
+  (via (at 111.25 76) (size 0.8) (drill 0.4) (layers F.Cu B.Cu) (net 2))
+  (via (at 109.75 74.75) (size 0.8) (drill 0.4) (layers F.Cu B.Cu) (net 2))
+  (via (at 105.25 80.25) (size 0.8) (drill 0.4) (layers F.Cu B.Cu) (net 1))
+  (via (at 108.25 80.25) (size 0.8) (drill 0.4) (layers F.Cu B.Cu) (net 1))
+  (via (at 106.75 80.25) (size 0.8) (drill 0.4) (layers F.Cu B.Cu) (net 1))
+  (via (at 105.25 82) (size 0.8) (drill 0.4) (layers F.Cu B.Cu) (net 1))
+  (via (at 108.25 82) (size 0.8) (drill 0.4) (layers F.Cu B.Cu) (net 1))
+  (via (at 106.75 82.25) (size 1.8) (drill 1.2) (layers F.Cu B.Cu) (net 1))
+  (via (at 106 81.125) (size 0.8) (drill 0.4) (layers F.Cu B.Cu) (net 1))
+  (via (at 107.5 81.125) (size 0.8) (drill 0.4) (layers F.Cu B.Cu) (net 1))
+  (via (at 112 81.125) (size 0.8) (drill 0.4) (layers F.Cu B.Cu) (net 2))
+  (via (at 109.75 82) (size 0.8) (drill 0.4) (layers F.Cu B.Cu) (net 2))
+  (via (at 110.5 81.125) (size 0.8) (drill 0.4) (layers F.Cu B.Cu) (net 2))
+  (via (at 112.75 80.25) (size 0.8) (drill 0.4) (layers F.Cu B.Cu) (net 2))
+  (via (at 109.75 80.25) (size 0.8) (drill 0.4) (layers F.Cu B.Cu) (net 2))
+  (via (at 111.25 80.25) (size 0.8) (drill 0.4) (layers F.Cu B.Cu) (net 2))
+  (via (at 112.75 82) (size 0.8) (drill 0.4) (layers F.Cu B.Cu) (net 2))
+  (via (at 111.25 82.25) (size 1.8) (drill 1.2) (layers F.Cu B.Cu) (net 2))
   (segment (start 106 88.5) (end 105 87.5) (width 0.4) (layer F.Cu) (net 1))
   (segment (start 107.575 88.5) (end 106 88.5) (width 0.4) (layer F.Cu) (net 1))
-  (segment (start 105 68) (end 105 75) (width 0.4) (layer F.Cu) (net 1))
   (segment (start 105.75 66.75) (end 105.75 65.75) (width 0.4) (layer F.Cu) (net 1))
   (segment (start 105.75 67.25) (end 105.75 66.75) (width 0.4) (layer F.Cu) (net 1))
   (segment (start 105 68) (end 105.75 67.25) (width 0.4) (layer F.Cu) (net 1))
+  (via (at 105.25 76) (size 0.8) (drill 0.4) (layers F.Cu B.Cu) (net 1))
+  (segment (start 105 68) (end 105 73.75) (width 0.4) (layer F.Cu) (net 1))
+  (segment (start 105 73.75) (end 105 75) (width 0.4) (layer F.Cu) (net 1))
+  (via (at 106.75 74.25) (size 1.8) (drill 1.2) (layers F.Cu B.Cu) (net 1))
   (segment (start 110.425 88.5) (end 112.25 88.5) (width 0.4) (layer F.Cu) (net 2))
   (segment (start 110 68.0625) (end 111.1875 68.0625) (width 0.4) (layer F.Cu) (net 2))
@@
   (segment (start 106.75 63) (end 109.6 63) (width 0.4) (layer F.Cu) (net 2))
   (segment (start 108 68.0625) (end 106.7875 68.0625) (width 0.4) (layer F.Cu) (net 2))
-  (segment (start 108 69.9375) (end 108 71) (width 0.4) (layer F.Cu) (net 3))
-  (segment (start 108 71) (end 109.5 72.5) (width 0.4) (layer F.Cu) (net 3))
-  (segment (start 109.5 72.5) (end 112 72.5) (width 0.4) (layer F.Cu) (net 3))
-  (segment (start 112 72.5) (end 113 71.5) (width 0.4) (layer F.Cu) (net 3))
-  (segment (start 113 71.5) (end 113 60.25) (width 0.4) (layer F.Cu) (net 3))
+  (via (at 111.25 74.25) (size 1.8) (drill 1.2) (layers F.Cu B.Cu) (net 2))
+  (segment (start 112.25 71.75) (end 113 71) (width 0.4) (layer F.Cu) (net 3))
+  (segment (start 108 70.75) (end 109 71.75) (width 0.4) (layer F.Cu) (net 3))
+  (segment (start 109 71.75) (end 112.25 71.75) (width 0.4) (layer F.Cu) (net 3))
+  (segment (start 113 71) (end 113 60.25) (width 0.4) (layer F.Cu) (net 3))
+  (segment (start 110.75 58) (end 106.75 58) (width 0.4) (layer F.Cu) (net 3))
   (segment (start 113 60.25) (end 110.75 58) (width 0.4) (layer F.Cu) (net 3))
-  (segment (start 110.75 58) (end 106.75 58) (width 0.4) (layer F.Cu) (net 3))
-  (segment (start 110.5 71.25) (end 110 70.75) (width 0.4) (layer F.Cu) (net 4))
-  (segment (start 112 70.75) (end 111.5 71.25) (width 0.4) (layer F.Cu) (net 4))
+  (segment (start 108 69.9375) (end 108 70.75) (width 0.4) (layer F.Cu) (net 3))
   (segment (start 110 70.75) (end 110 69.9375) (width 0.4) (layer F.Cu) (net 4))
-  (segment (start 111.5 71.25) (end 110.5 71.25) (width 0.4) (layer F.Cu) (net 4))
+  (segment (start 110.25 71) (end 110 70.75) (width 0.4) (layer F.Cu) (net 4))
+  (segment (start 111.75 71) (end 110.25 71) (width 0.4) (layer F.Cu) (net 4))
+  (segment (start 112 70.75) (end 111.75 71) (width 0.4) (layer F.Cu) (net 4))
   (segment (start 112 61.5) (end 112 70.75) (width 0.4) (layer F.Cu) (net 4))
   (segment (start 111 60.5) (end 112 61.5) (width 0.4) (layer F.Cu) (net 4))
@@
     (polygon
       (pts
-        (xy 104.7 76.75) (xy 104.725 74) (xy 108.775 74) (xy 108.75 76.75)
+        (xy 104.75 76.75) (xy 104.75 73) (xy 108 73) (xy 108.75 73.75) (xy 108.75 76.75)
       )
     )
@@
     (polygon
       (pts
-        (xy 113.3 74.25) (xy 113.3 76.75) (xy 109.15 76.75) (xy 109.15 74.25)
+        (xy 113.3 73) (xy 113.3 76.75) (xy 109.15 76.75) (xy 109.15 73)
       )
     )

Commit message: Export rev F
Routing:
- added copper zone on B.Cu, net +5V
- added copper zone on B.Cu, net /Photodiode
Changed lines of the file:
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@@
   (general
     (thickness 1.6)
-    (drawings 46)
+    (drawings 49)
     (tracks 60)
     (zones 0)
@@
     (visible_elements FFFFFF7F)
     (pcbplotparams
-      (layerselection 0x210a8_7fffffff)
+      (layerselection 0x310fc_ffffffff)
       (usegerberextensions false)
       (usegerberattributes false)
@@
     )
   )
+  (dimension 20.4 (width 0.15) (layer Margin)
+    (gr_text "20.400 mm" (at 120.55 66.7 90) (layer Margin)
+      (effects (font (size 1 1) (thickness 0.15)))
+    )
+    (feature1 (pts (xy 114 56.5) (xy 119.836421 56.5)))
+    (feature2 (pts (xy 114 76.9) (xy 119.836421 76.9)))
+    (crossbar (pts (xy 119.25 76.9) (xy 119.25 56.5)))
+    (arrow1a (pts (xy 119.25 56.5) (xy 119.836421 57.626504)))
+    (arrow1b (pts (xy 119.25 56.5) (xy 118.663579 57.626504)))
+    (arrow2a (pts (xy 119.25 76.9) (xy 119.836421 75.773496)))
+    (arrow2b (pts (xy 119.25 76.9) (xy 118.663579 75.773496)))
+  )
+  (dimension 14 (width 0.15) (layer Margin)
+    (gr_text "14.000 mm" (at 120.55 86 90) (layer Margin)
+      (effects (font (size 1 1) (thickness 0.15)))
+    )
+    (feature1 (pts (xy 114 79) (xy 119.836421 79)))
+    (feature2 (pts (xy 114 93) (xy 119.836421 93)))
+    (crossbar (pts (xy 119.25 93) (xy 119.25 79)))
+    (arrow1a (pts (xy 119.25 79) (xy 119.836421 80.126504)))
+    (arrow1b (pts (xy 119.25 79) (xy 118.663579 80.126504)))
+    (arrow2a (pts (xy 119.25 93) (xy 119.836421 91.873496)))
+    (arrow2b (pts (xy 119.25 93) (xy 118.663579 91.873496)))
+  )
+  (dimension 10 (width 0.15) (layer Margin)
+    (gr_text "10.000 mm" (at 109 97.55) (layer Margin)
+      (effects (font (size 1 1) (thickness 0.15)))
+    )
+    (feature1 (pts (xy 114 93) (xy 114 96.836421)))
+    (feature2 (pts (xy 104 93) (xy 104 96.836421)))
+    (crossbar (pts (xy 104 96.25) (xy 114 96.25)))
+    (arrow1a (pts (xy 114 96.25) (xy 112.873496 96.836421)))
+    (arrow1b (pts (xy 114 96.25) (xy 112.873496 95.663579)))
+    (arrow2a (pts (xy 104 96.25) (xy 105.126504 96.836421)))
+    (arrow2b (pts (xy 104 96.25) (xy 105.126504 95.663579)))
+  )
   (gr_text +5V (at 109.25 63) (layer F.SilkS)
     (effects (font (size 0.8 0.8) (thickness 0.15)) (justify left))
@@
   (via (at 107.5 75.375) (size 0.8) (drill 0.4) (layers F.Cu B.Cu) (net 1))
   (via (at 106 75.375) (size 0.8) (drill 0.4) (layers F.Cu B.Cu) (net 1))
-  (via (at 112 75.375) (size 0.8) (drill 0.4) (layers F.Cu B.Cu) (net 2))
-  (via (at 109.75 76) (size 0.8) (drill 0.4) (layers F.Cu B.Cu) (net 2))
-  (via (at 112.75 74.75) (size 0.8) (drill 0.4) (layers F.Cu B.Cu) (net 2))
-  (via (at 112.75 76) (size 0.8) (drill 0.4) (layers F.Cu B.Cu) (net 2))
-  (via (at 110.5 75.375) (size 0.8) (drill 0.4) (layers F.Cu B.Cu) (net 2))
-  (via (at 111.25 76) (size 0.8) (drill 0.4) (layers F.Cu B.Cu) (net 2))
-  (via (at 109.75 74.75) (size 0.8) (drill 0.4) (layers F.Cu B.Cu) (net 2))
   (via (at 105.25 80.25) (size 0.8) (drill 0.4) (layers F.Cu B.Cu) (net 1))
   (via (at 108.25 80.25) (size 0.8) (drill 0.4) (layers F.Cu B.Cu) (net 1))
@@
   (via (at 106 81.125) (size 0.8) (drill 0.4) (layers F.Cu B.Cu) (net 1))
   (via (at 107.5 81.125) (size 0.8) (drill 0.4) (layers F.Cu B.Cu) (net 1))
-  (via (at 112 81.125) (size 0.8) (drill 0.4) (layers F.Cu B.Cu) (net 2))
-  (via (at 109.75 82) (size 0.8) (drill 0.4) (layers F.Cu B.Cu) (net 2))
-  (via (at 110.5 81.125) (size 0.8) (drill 0.4) (layers F.Cu B.Cu) (net 2))
-  (via (at 112.75 80.25) (size 0.8) (drill 0.4) (layers F.Cu B.Cu) (net 2))
-  (via (at 109.75 80.25) (size 0.8) (drill 0.4) (layers F.Cu B.Cu) (net 2))
-  (via (at 111.25 80.25) (size 0.8) (drill 0.4) (layers F.Cu B.Cu) (net 2))
-  (via (at 112.75 82) (size 0.8) (drill 0.4) (layers F.Cu B.Cu) (net 2))
-  (via (at 111.25 82.25) (size 1.8) (drill 1.2) (layers F.Cu B.Cu) (net 2))
   (segment (start 106 88.5) (end 105 87.5) (width 0.4) (layer F.Cu) (net 1))
   (segment (start 107.575 88.5) (end 106 88.5) (width 0.4) (layer F.Cu) (net 1))
@@
   (segment (start 105 73.75) (end 105 75) (width 0.4) (layer F.Cu) (net 1))
   (via (at 106.75 74.25) (size 1.8) (drill 1.2) (layers F.Cu B.Cu) (net 1))
+  (via (at 112 75.375) (size 0.8) (drill 0.4) (layers F.Cu B.Cu) (net 2))
+  (via (at 109.75 76) (size 0.8) (drill 0.4) (layers F.Cu B.Cu) (net 2))
+  (via (at 112.75 74.75) (size 0.8) (drill 0.4) (layers F.Cu B.Cu) (net 2))
+  (via (at 112.75 76) (size 0.8) (drill 0.4) (layers F.Cu B.Cu) (net 2))
+  (via (at 110.5 75.375) (size 0.8) (drill 0.4) (layers F.Cu B.Cu) (net 2))
+  (via (at 111.25 76) (size 0.8) (drill 0.4) (layers F.Cu B.Cu) (net 2))
+  (via (at 109.75 74.75) (size 0.8) (drill 0.4) (layers F.Cu B.Cu) (net 2))
+  (via (at 112 81.125) (size 0.8) (drill 0.4) (layers F.Cu B.Cu) (net 2))
+  (via (at 109.75 82) (size 0.8) (drill 0.4) (layers F.Cu B.Cu) (net 2))
+  (via (at 110.5 81.125) (size 0.8) (drill 0.4) (layers F.Cu B.Cu) (net 2))
+  (via (at 112.75 80.25) (size 0.8) (drill 0.4) (layers F.Cu B.Cu) (net 2))
+  (via (at 109.75 80.25) (size 0.8) (drill 0.4) (layers F.Cu B.Cu) (net 2))
+  (via (at 111.25 80.25) (size 0.8) (drill 0.4) (layers F.Cu B.Cu) (net 2))
+  (via (at 112.75 82) (size 0.8) (drill 0.4) (layers F.Cu B.Cu) (net 2))
+  (via (at 111.25 82.25) (size 1.8) (drill 1.2) (layers F.Cu B.Cu) (net 2))
   (segment (start 110.425 88.5) (end 112.25 88.5) (width 0.4) (layer F.Cu) (net 2))
   (segment (start 110 68.0625) (end 111.1875 68.0625) (width 0.4) (layer F.Cu) (net 2))
@@
       )
     )
+  )
+  (zone (net 1) (net_name /Photodiode) (layer B.Cu) (hatch edge 0.508)
+    (priority 1)
+    (connect_pads no (clearance 0))
+    (min_thickness 0.25)
+    (fill yes (arc_segments 32) (thermal_gap 0.508) (thermal_bridge_width 0.508))
+    (polygon
+      (pts
+        (xy 104.75 76.75) (xy 104.75 73) (xy 108 73) (xy 108.75 73.75) (xy 108.75 76.75)
+      )
+    )
+  )
+  (zone (net 2) (net_name +5V) (layer B.Cu) (hatch edge 0.508)
+    (connect_pads no (clearance 0))
+    (min_thickness 0.25)
+    (fill yes (arc_segments 32) (thermal_gap 0.508) (thermal_bridge_width 0.508))
+    (polygon
+      (pts
+        (xy 113.3 73) (xy 113.3 76.75) (xy 109.15 76.75) (xy 109.15 73)
+      )
+    )
+  )
+  (zone (net 2) (net_name +5V) (layer B.Cu) (hatch edge 0.508)
+    (connect_pads no (clearance 0.4))
+    (min_thickness 0.25)
+    (fill yes (arc_segments 32) (thermal_gap 0.508) (thermal_bridge_width 0.508))
+    (polygon
+      (pts
+        (xy 104 76.9) (xy 114 76.9) (xy 114 56.5) (xy 104 56.5)
+      )
+    )
+  )
+  (zone (net 2) (net_name +5V) (layer B.Cu) (hatch edge 0.508)
+    (connect_pads no (clearance 0.4))
+    (min_thickness 0.25)
+    (fill yes (arc_segments 32) (thermal_gap 0.508) (thermal_bridge_width 0.508))
+    (polygon
+      (pts
+        (xy 109.25 93) (xy 114 93) (xy 114 79) (xy 109.25 79)
+      )
+    )
+  )
+  (zone (net 1) (net_name /Photodiode) (layer B.Cu) (hatch edge 0.508)
+    (connect_pads no (clearance 0.4))
+    (min_thickness 0.25)
+    (fill yes (arc_segments 32) (thermal_gap 0.508) (thermal_bridge_width 0.508))
+    (polygon
+      (pts
+        (xy 104 79) (xy 108.5 79) (xy 108.75 79) (xy 108.75 93) (xy 104 93)
+      )
+    )

Commit message: Rev G
Parts:
- added FID1: Fiducial, Fiducial:Fiducial_0.5mm_Mask1mm, F.Cu at (105.0, 84.2)
- added FID2: Fiducial, Fiducial:Fiducial_0.5mm_Mask1mm, F.Cu at (113.0, 86.2)
- added FID3: Fiducial, Fiducial:Fiducial_0.5mm_Mask1mm, F.Cu at (105.9, 64.2)
- added FID4: Fiducial, Fiducial:Fiducial_0.5mm_Mask1mm, F.Cu at (113.0, 69.8)
- added G***: LOGO, POxiM-logos:POxiMLogo_GoldHeart_W5mm, F.Cu at (107.0, 71.8)
- added H1: M2 alignment hole, MountingHole:MountingHole_2.2mm_M2, F.Cu at (106.0, 88.0)
- added H2: M2 alignment hole, MountingHole:MountingHole_2.2mm_M2, F.Cu at (112.0, 88.0)
- added H3: M2 alignment hole, MountingHole:MountingHole_2.2mm_M2, F.Cu at (112.2, 64.8)
- added H4: M2 alignment hole, MountingHole:MountingHole_2.2mm_M2, F.Cu at (112.2, 71.5)
- D1: footprint LED_SMD:LED_1206_3216Metric_Castellated -> POxiM-uncategorised:LED_1206_3216Metric_0805_2012Metric_Castellated
- D2, D3: footprint LED_SMD:LED_0805_2012Metric -> POxiM-uncategorised:LED_0805_2012Metric_0603_1608Metric
- G***, J3: moved to B.Cu
- moved J3 6.25 mm to (106.8, 68.0), turned to 180 degrees
- moved G*** 5.75 mm to (109.0, 85.2)
- moved D1 3.00 mm to (109.0, 85.5), turned to 0 degrees
Connections:
- D1 pad 1: +5V -> /Photodiode
- D1 pad 2: /Photodiode -> GND
- D2 pad 1: /LED.IR -> GND
- D2 pad 2: +5V -> /LED.IR
- D3 pad 1: /LED.Red -> GND
- D3 pad 2: +5V -> /LED.Red
- J3 pad 1: /LED.IR -> /LED.Red
- J3 pad 2: /LED.Red -> /LED.IR
- J3 pad 3: +5V -> GND
Routing:
- net /LED.IR: track 24.5 -> 1.58 mm, vias 0 -> 6
- net /LED.Red: track 17.9 -> 4.82 mm, vias 0 -> 6
- net +5V: track 11.3 -> 0.00 mm, vias 16 -> 0
- net /Photodiode: track 12.5 -> 5.33 mm, vias 16 -> 22
- net GND: track 0.00 -> 6.96 mm, vias 0 -> 23
- added copper zone on F.Cu, net /LED.Red
- added copper zone on B.Cu, net GND
- added copper zone on F.Cu, net GND
- removed copper zone on B.Cu, net +5V
- removed copper zone on F.Cu, net +5V
Other:
- board size 10 x 36.5 mm -> 10 x 27.2 mm
- board text added: "Finger sensor Rev G"
- board text added: "GND"
- board text removed: "+5V"
- board text removed: "Finger sensor Rev F"
