File: POxiM-fingersensor.kicad_pcb (KiCad board)
At the start: 2 copper layers, 10 x 27.2 mm, 14 parts, among them J3 To readout unit

Commit message: Rev H
Parts:
- moved H3 0.90 mm to (111.5, 65.2)
- moved H4 0.75 mm to (111.5, 71.5)
- moved H1 0.71 mm to (106.5, 87.5)
- moved H2 0.71 mm to (111.5, 87.5)
- moved D1 0.50 mm to (109.0, 86.0), turned to 270 degrees
- moved G*** 0.25 mm to (109.0, 85.0)
Routing:
- net GND: track 6.96 -> 8.87 mm
Other:
- board text added: "Finger sensor Rev H"
- board text removed: "Finger sensor Rev G"

Commit message: Rev I
Parts:
- FID1, FID2, FID3, FID4: footprint Fiducial:Fiducial_0.5mm_Mask1mm -> POxiM-uncategorised:Fiducial_1mm_Mask2mm
- H1, H2, H3, H4: footprint MountingHole:MountingHole_2.2mm_M2 -> POxiM-uncategorised:AlignmentHole_2mm
- moved G*** 17.5 mm to (109.0, 89.1)
- moved D2 1.50 mm to (108.0, 70.5)
- moved D3 1.50 mm to (110.0, 70.5)
- moved FID1 1.35 mm to (105.5, 85.5)
- moved FID2 0.90 mm to (112.5, 85.5)
- moved H4 0.75 mm to (112.2, 71.5)
- moved FID4 0.71 mm to (112.5, 69.2)
- moved D1 0.60 mm to (109.0, 85.4), turned to 0 degrees
- moved FID3 0.42 mm to (106.3, 64.2)
Routing:
- net /Photodiode: track 5.69 -> 8.26 mm, vias 22 -> 21
- net /LED.Red: track 4.82 -> 6.23 mm
- net /LED.IR: track 1.58 -> 2.91 mm
- net GND: track 8.87 -> 9.95 mm, vias 23 -> 24
Other:
- board text added: "Fingsens"
- board text added: "Rev I"
- board text removed: "Finger sensor Rev H"

Commit message: Rev J
Parts:
- removed the G*** at (109.0, 89.1)
- added G***: LOGO, POxiM-logos:POxiMLogo_GoldHeart_W7_5mm, F.Cu at (109.0, 92.2)
- moved FID1 4.50 mm to (105.5, 90.0)
- moved H1 2.51 mm to (106.8, 85.0)
- moved H2 2.26 mm to (111.2, 89.8)
- moved G*** 2.25 mm to (109.0, 87.2)
- moved D1 1.60 mm to (109.0, 87.0), turned to 270 degrees
- moved FID2 0.75 mm to (112.5, 84.8)
- moved FID3 0.50 mm to (106.3, 63.8)
- moved J3 0.50 mm to (106.8, 67.5)
Routing:
- net GND: track 9.95 -> 6.38 mm, vias 24 -> 23
Other:
- board size 10 x 27.2 mm -> 10 x 31.1 mm
- net class Default: clearance 0.2 -> 0.4; trace_width 0.2 -> 0.4
- rule trace_clearance: 0.2 -> 0.4
- rule trace_min: 0.2 -> 0.4
- board text added: "Rev J"
- board text removed: "Rev I"

Commit message: Rev K
Parts:
- moved D1 2.10 mm to (109.0, 89.1)
- moved D2 2.10 mm to (108.0, 68.4)
- moved D3 2.10 mm to (110.0, 68.4)
- moved FID2 1.25 mm to (111.8, 85.8)
- moved H2 0.50 mm to (111.2, 89.2)
Routing:
- net /LED.Red: track 6.23 -> 4.13 mm
- net /Photodiode: track 8.22 -> 10.3 mm, vias 21 -> 24
- net /LED.IR: track 2.91 -> 1.42 mm
Other:
- board text added: "Rev K"
- board text removed: "Rev J"
