File: POxiM-fingersensor-PhotoDiodeBoard.kicad_pcb (KiCad board)
At the start: 2 copper layers, 10 x 31.1 mm, 14 parts, among them J3 To readout unit

Commit message: Rev K
Parts:
- removed D2: IR (940nm), POxiM-uncategorised:LED_0805_2012Metric_0603_1608Metric
- removed D3: Red (660nm), POxiM-uncategorised:LED_0805_2012Metric_0603_1608Metric
- removed FID3, FID4: Fiducial, POxiM-uncategorised:Fiducial_1mm_Mask2mm
- removed H3, H4: M2 alignment hole, POxiM-uncategorised:AlignmentHole_2mm
- removed J3: To readout unit, POxiM-uncategorised:Finger-CableConnection
Routing:
- net GND: track 6.64 -> 1.89 mm, vias 23 -> 8
- net /LED.Red: track 4.13 -> 0.00 mm, vias 6 -> 0
- net /Photodiode: track 10.3 -> 6.57 mm, vias 24 -> 8
- net /LED.IR: track 1.42 -> 0.00 mm, vias 6 -> 0
- removed copper zone on F.Cu, net /LED.IR
- removed copper zone on F.Cu, net /LED.Red
Other:
- board size 10 x 31.1 mm -> 10 x 14.5 mm
- board text removed: "Fingsens"
- board text removed: "GND"
- board text removed: "IR"
- board text removed: "PD"
- board text removed: "Red"
- board text removed: "Rev H"
